Commit message: plus de ik

File: pincher_arm/pincher_arm_description/urdf/mod.xacro (robot description, xacro)
@@ -57,5 +57,5 @@
     <!-- shoulder pan joint -->
     <xacro:dynamixel_AX12_fixed parent="arm_base_link" name="arm_shoulder_pan_servo">
-      <origin xyz="0.1 0 0.0555" rpy="${pi/2} 0 ${pi/2}"/>
+      <origin xyz="0.1 0 0.055" rpy="${pi/2} 0 ${pi/2}"/>
     </xacro:dynamixel_AX12_fixed>
     <xacro:bioloid_F3_revolute parent="arm_shoulder_pan_servo_link" name="arm_shoulder_pan" color="${color}"
@@ -170,14 +170,15 @@
     <link name="chassis_link">
             <visual>
-                <origin rpy="0 0 0" xyz="-0.027 -0.2445 -0.07"/>
-                <geometry>
-                    <mesh scale="0.001 0.001 0.001" filename="package://wifibot_arm_description/meshes/box_wifibot.stl"/>
-                </geometry>
-                <material name="Gray"/>
-            </visual>
-            <collision>
-                <origin rpy="0 0 0" xyz="0 -0.2445 -0.07"/>
-                <geometry>
-                    <mesh scale="0.001 0.001 0.001" filename="package://wifibot_arm_description/meshes/box_wifibot.stl"/>
+                <origin rpy="0 0 0" xyz="0.13 0 0"/>
+                <geometry>
+                    <box size="0.26 0.2 0.08"/>
+                </geometry>
+                <material name="black"/>
+            </visual>
+            <collision>
+                <origin rpy="0 0 0" xyz="0 0 0.06"/>
+                <geometry>
+                    <!--mesh scale="0.001 0.001 0.001" filename="package://manipulator_description/meshes/bow_wifibot.stl"/>-->
+                    <box size="0.26 0.2 0.08"/>
                 </geometry>
             </collision>
@@ -197,15 +198,15 @@
             </inertial>
             <collision>
-                <origin rpy="-1.570796 0 0" xyz="0 0 0.045"/>
-                <geometry>
-                    <mesh scale="0.418 0.6 0.418 " filename="package://wifibot_arm_description/meshes/wheel_smb.dae"/>
-                </geometry>
-            </collision>
-            <visual>
-                <origin rpy="-1.570796 0 0" xyz="0 0 0.045"/>
-                <geometry>
-                    <mesh scale="0.418 0.6 0.418 " filename="package://wifibot_arm_description/meshes/wheel_smb.dae"/>
-                </geometry>
-                <material name="Gray"/>
+                <origin rpy="-1.570796 0 0" xyz="0 0 0.040"/>
+                <geometry>
+                    <mesh scale="0.418 0.6 0.418 " filename="package://wifibot_arm_description/meshes/wheel_smb.dae"/>
+                </geometry>
+            </collision>
+            <visual>
+                <origin rpy="-1.570796 0 0" xyz="0 0 0.040"/>
+                <geometry>
+                    <mesh scale="0.418 0.6 0.418 " filename="package://wifibot_arm_description/meshes/wheel_smb.dae"/>
+                </geometry>
+                <material name="gray"/>
             </visual>
     </link>
@@ -224,15 +225,15 @@
             </inertial>
             <collision>
-                <origin rpy="1.570796 0 0" xyz="0 0 0.045"/>
-                <geometry>
-                    <mesh scale="0.418 0.6 0.418 " filename="package://wifibot_arm_description/meshes/wheel_smb.dae"/>
-                </geometry>
-            </collision>
-            <visual>
-                <origin rpy="1.570796 0 0" xyz="0 0 0.045"/>
-                <geometry>
-                    <mesh scale="0.418 0.6 0.418 " filename="package://wifibot_arm_description/meshes/wheel_smb.dae"/>
-                </geometry>
-                <material name="Gray"/>
+                <origin rpy="1.570796 0 0" xyz="0 0 0.040"/>
+                <geometry>
+                    <mesh scale="0.418 0.6 0.418 " filename="package://wifibot_arm_description/meshes/wheel_smb.dae"/>
+                </geometry>
+            </collision>
+            <visual>
+                <origin rpy="1.570796 0 0" xyz="0 0 0.040"/>
+                <geometry>
+                    <mesh scale="0.418 0.6 0.418 " filename="package://wifibot_arm_description/meshes/wheel_smb.dae"/>
+                </geometry>
+                <material name="gray"/>
             </visual>
     </link>
@@ -251,15 +252,15 @@
             </inertial>
             <collision>
-                <origin rpy="-1.570796 0 0" xyz="0 0 0.045"/>
-                <geometry>
-                    <mesh scale="0.418 0.6 0.418 " filename="package://wifibot_arm_description/meshes/wheel_smb.dae"/>
-                </geometry>
-            </collision>
-            <visual>
-                <origin rpy="-1.570796 0 0" xyz="0 0 0.045"/>
-                <geometry>
-                    <mesh scale="0.418 0.6 0.418 " filename="package://wifibot_arm_description/meshes/wheel_smb.dae"/>
-                </geometry>
-                <material name="Gray"/>
+                <origin rpy="-1.570796 0 0" xyz="0 0 0.040"/>
+                <geometry>
+                    <mesh scale="0.418 0.6 0.418 " filename="package://wifibot_arm_description/meshes/wheel_smb.dae"/>
+                </geometry>
+            </collision>
+            <visual>
+                <origin rpy="-1.570796 0 0" xyz="0 0 0.040"/>
+                <geometry>
+                    <mesh scale="0.418 0.6 0.418 " filename="package://wifibot_arm_description/meshes/wheel_smb.dae"/>
+                </geometry>
+                <material name="gray"/>
             </visual>
     </link>
@@ -278,15 +279,15 @@
             </inertial>
             <collision>
-                <origin rpy="1.570796 0 0" xyz="0 0 0.045"/>
-                <geometry>
-                    <mesh scale="0.418 0.6 0.418 " filename="package://wifibot_arm_description/meshes/wheel_smb.dae"/>
-                </geometry>
-            </collision>
-            <visual>
-                <origin rpy="1.570796 0 0" xyz="0 0 0.045"/>
-                <geometry>
-                    <mesh scale="0.418 0.6 0.418 " filename="package://wifibot_arm_description/meshes/wheel_smb.dae"/>
-                </geometry>
-                <material name="Gray"/>
+                <origin rpy="1.570796 0 0" xyz="0 0 0.040"/>
+                <geometry>
+                    <mesh scale="0.418 0.6 0.418 " filename="package://wifibot_arm_description/meshes/wheel_smb.dae"/>
+                </geometry>
+            </collision>
+            <visual>
+                <origin rpy="1.570796 0 0" xyz="0 0 0.040"/>
+                <geometry>
+                    <mesh scale="0.418 0.6 0.418 " filename="package://wifibot_arm_description/meshes/wheel_smb.dae"/>
+                </geometry>
+                <material name="gray"/>
             </visual>
     </link>
